Commit message: 20200229
ディレクトリ構造の見直しと、ファイル名および、launchファイルの整理

File: seto_scararobot_description/urdf/seto_scararobot.urdf (robot description, URDF)
Before this commit: robot seto_scararobot, 4 links, 3 joints
Links:
- added link world
- link arm1_link: mass None -> 0.042; geometry visual mesh filename=package://seto_scararobot_description/meshes/arm1.stl
- link arm2_link: mass None -> 0.221; geometry visual mesh filename=package://seto_scararobot_description/meshes/arm2.stl
- link base_link: mass None -> 2.935; geometry visual mesh filename=package://seto_scararobot_description/meshes/base.stl
- link endpoint: mass None -> 0; geometry visual mesh filename=package://seto_scararobot_description/meshes/endpoint.stl
Joints:
- added joint fixed: type fixed, parent world, child base_link

Commit message: 20200308
seto_scara_gazebo_moveitを作成

File: seto_scararobot_description/urdf/seto_scararobot.urdf (robot description, URDF)
Before this commit: robot seto_scararobot, 5 links, 4 joints
Links:
- link arm1_link: geometry collision mesh filename=package://seto_scararobot_description/meshes/arm1.stl; visual mesh filename=package://seto_scararobot_description/meshes/arm1.stl
- link arm2_link: geometry collision mesh filename=package://seto_scararobot_description/meshes/arm2.stl; visual mesh filename=package://seto_scararobot_description/meshes/arm2.stl
- link base_link: geometry collision mesh filename=package://seto_scararobot_description/meshes/base.stl; visual mesh filename=package://seto_scararobot_description/meshes/base.stl
- link endpoint: mass 0 -> 0.001; geometry 
Joints:
- removed joint fixed
- added joint fixed_world: type fixed, parent world, child base_link

Commit message: 20200320

File: seto_scararobot_description/urdf/seto_scararobot.urdf (robot description, URDF)
Before this commit: robot seto_scararobot, 5 links, 4 joints
Joints:
- joint arm1_to_arm2: limit lower=-3.14159 upper=3.14159 effort=1000.0 velocity=0.5 -> lower=-3.14159 upper=3.14159 effort=1000.0 velocity=3.0
- joint base_to_arm1: limit lower=-3.14159 upper=3.14159 effort=1000.0 velocity=0.5 -> lower=-3.14159 upper=3.14159 effort=1000.0 velocity=3.0
- joint end_joint: limit lower=-3.14159 upper=3.14159 effort=1000.0 velocity=0.5 -> lower=-3.14159 upper=3.14159 effort=1000.0 velocity=3.0
